File: module_LoRa_Kicad/RN2483shield.kicad_pcb (KiCad board)
At the start: 2 copper layers, 53.2 x 30.6 mm, 9 parts, among them J1 Screw_Terminal_01x04, J2 SMA_HF, J3 Screw_Terminal_01x03, U1 RN2483/RN2903

Commit message: 27/11/2023
Parts:
- moved J3 9.06 mm to (206.1, 75.6)
- moved J2 5.55 mm to (216.7, 95.9)
- moved U1 3.24 mm to (174.5, 77.0)
- moved R3 2.19 mm to (183.5, 98.4)
- moved R2 2.19 mm to (187.5, 98.4)
Routing:
- net GND: track 109.0 -> 0.00 mm, vias 43 -> 58
- net PGC_INT: track 9.07 -> 22.0 mm
- net PGD_INT: track 7.95 -> 19.9 mm
- net RESET: track 31.3 -> 42.6 mm
- net TX_RADIO: track 30.2 -> 20.2 mm
- net Net-(J2-RF): track 10.4 -> 17.8 mm
- net RX_RADIO: track 60.1 -> 55.2 mm
- net +3V3: track 63.8 -> 63.1 mm
Other:
- board size 53.2 x 30.6 mm -> 53.1 x 30.6 mm
- board text added: "GEII Corp. LoRa"
- board text added: "GEII Corp. LoRa V2"
- board text added: "电气工程和工业计算机"
- board text removed: "GEII Corp. LoRa V1"
